Commit message: Update

File: hunter_robot/urdf/mid360.xacro (robot description, xacro)
@@ -23,4 +23,5 @@
 <xacro:box_inertia m="${length}" w="${width}" d="${length}" h="${height}"/>
   <visual>
+        <origin xyz="0.025 -0.0265 -0.025" rpy="${pi/2} 0 ${pi}"/>
         <geometry>
             <!-- <box size="${length} ${width} ${height}"/> -->
