Commit message: 双轮差速完成

File: hunter_robot/urdf/diff.urdf (robot description, URDF)
Before this commit: robot robot, 6 links, 5 joints
Links:
- removed link base_footprint
Joints:
- removed joint base_joint

File: hunter_robot/urdf/mid360.xacro (robot description, xacro)
@@ -4,5 +4,5 @@
   <xacro:property name="laser_min_range" value="0.1"/>
   <xacro:property name="laser_max_range" value="200.0"/>
-  <xacro:property name="samples" value="40000"/>
+  <xacro:property name="samples" value="30000"/>
   <xacro:property name="resolution" value="0.002"/>
   <xacro:property name="noise_mean" value="0.0"/>
