Commit message: Update

File: hunter_robot/urdf/diff.xacro (robot description, xacro)
@@ -246,6 +246,6 @@
   <!-- Livox-Mid360  -->
   <xacro:include filename="$(find hunter_robot)/urdf/mid360.xacro" />
-  <xacro:mid360 name="livox_frame" parent="base_link" topic="/livox/lidar">
-    <origin xyz="0 0 0.135" rpy="0 0 0" />
+  <xacro:mid360 name="livox_frame" mid360_link="base_link" topic="/livox/lidar">
+    <origin xyz="0 0 -0.135" rpy="0 0 0" />
   </xacro:mid360>
 </robot>

File: hunter_robot/urdf/mecanum.xacro (robot description, xacro)
@@ -12,7 +12,6 @@
   </xacro:macro>
   <!-- base_link to livox_frame -->
-  <xacro:arg name="xyz" default="0.12 0.0 0.175" />
+  <xacro:arg name="xyz" default="-0.12 0.0 -0.175" />
   <xacro:arg name="rpy" default="0 0 0" />
-  <link name="dummy"/>
   <link name="base_link">
     <visual>
@@ -33,8 +32,4 @@
     <xacro:default_inertial mass="8.2"/>
   </link>
-  <joint name="dummy_joint" type="fixed">
-     <parent link="dummy"/>
-     <child link="base_link"/>
-  </joint>
   <link name="wheel_1">
     <visual>
@@ -229,5 +224,5 @@
   <!-- Livox-Mid360  -->
   <xacro:include filename="$(find hunter_robot)/urdf/mid360.xacro" />
-  <xacro:mid360 name="livox_frame" parent="base_link" topic="/livox/lidar">
+  <xacro:mid360 name="livox_frame" mid360_link="base_link" topic="/livox/lidar">
     <origin xyz="$(arg xyz)" rpy="$(arg rpy)" />
   </xacro:mid360>

File: hunter_robot/urdf/mid360.xacro (robot description, xacro)
@@ -19,5 +19,5 @@
     </inertial>
   </xacro:macro>
-  <xacro:macro name="mid360" params="name:='' parent:= 'base_link' topic:='mid360' *origin ">
+  <xacro:macro name="mid360" params="name:='' mid360_link:= 'base_link' topic:='mid360' *origin ">
 <link name="${name}">
 <xacro:box_inertia m="${length}" w="${width}" d="${length}" h="${height}"/>
@@ -31,6 +31,6 @@
 </link>
     <joint name="${name}_joint" type="fixed">
-      <parent link="${parent}"/>
-      <child link="${name}"/>
+      <parent link="${name}"/>
+      <child link="${mid360_link}"/>
       <xacro:insert_block name="origin"/>
     </joint>
